Commit message: added hardware documentation

File: adsmt_description/adsmt_description/urdf/adsmt.xacro (robot description, xacro)
@@ -6,16 +6,16 @@
     </link>
     <joint name = "body_link_joint" type='fixed'>
-        <origin xyz="0 0 0.5" rpy="0 0 0"/>
+        <origin xyz="0 0 1.5" rpy="0 0 0"/>
         <parent link="base_footprint"/>
         <child link="body"/>
     </joint>
     <material name="yellow">
-        <color rgba="1 1 0 1"/>
+        <color rgba="1 0.5 0 1"/>
     </material>
     <material name="black">
-        <color rgba="0 0 0 1"/>
+        <color rgba="0.02 0.02 0.02 1"/>
     </material>
-    <material name="blue">
-        <color rgba="0 0 1 1"/>
+    <material name="grey">
+        <color rgba="0.06 0.06 0.06 1"/>
     </material>
     <!-- Base Link -->
@@ -30,6 +30,5 @@
                 <mesh filename="$(find adsmt_description)/adsmt_description/urdf/designs/body.stl" scale=" 0.01 0.01 0.01"/>
             </geometry>
-            <material name='black'>
-            </material>
+            <material name='grey'/>
         </visual>
             <collision>
@@ -58,7 +57,6 @@
             <geometry>
                 <mesh filename="$(find adsmt_description)/adsmt_description/urdf/designs/double_u.stl" scale=" 0.01 0.01 0.01"/>
-            <material name='yellow'>
-            </material>
-            </geometry>
+            </geometry>
+            <material name='yellow'/>
         </visual>
         <collision>
@@ -85,6 +83,6 @@
             <geometry>
                 <mesh filename="$(find adsmt_description)/adsmt_description/urdf/designs/thigh.stl" scale=" 0.01 0.01 0.01"/>
+            </geometry>
             <material name='black'></material>
-            </geometry>
         </visual>
             <collision>
@@ -112,6 +110,6 @@
             <geometry>
                 <mesh filename="$(find adsmt_description)/adsmt_description/urdf/designs/shin.stl" scale=" 0.01 0.01 0.01"/>
-            <material name='yellow'></material>
-            </geometry>
+            </geometry>
+            <material name='yellow'></material>
         </visual>
             <collision>
@@ -139,6 +137,6 @@
             <geometry>
                 <mesh filename="$(find adsmt_description)/adsmt_description/urdf/designs/double_u_r.stl" scale=" 0.01 0.01 0.01"/>
-            <material name='yellow'></material>
-            </geometry>
+            </geometry>
+            <material name='yellow'/>
         </visual>
             <collision>
@@ -165,6 +163,6 @@
             <geometry>
                 <mesh filename="$(find adsmt_description)/adsmt_description/urdf/designs/thigh.stl" scale=" 0.01 0.01 0.01"/>
+            </geometry>
             <material name='black'></material>
-            </geometry>
         </visual>
             <collision>
@@ -191,6 +189,6 @@
             <geometry>
                 <mesh filename="$(find adsmt_description)/adsmt_description/urdf/designs/shin.stl" scale=" 0.01 0.01 0.01"/>
-            <material name='yellow'></material>
-            </geometry>
+            </geometry>
+            <material name='yellow'></material>
         </visual>
             <collision>
@@ -218,6 +216,6 @@
             <geometry>
                 <mesh filename="$(find adsmt_description)/adsmt_description/urdf/designs/double_u.stl" scale=" 0.01 0.01 0.01"/>
-            <material name='yellow'></material>
-            </geometry>
+            </geometry>
+            <material name='yellow'></material>
         </visual>
             <collision>
@@ -244,6 +242,6 @@
             <geometry>
                 <mesh filename="$(find adsmt_description)/adsmt_description/urdf/designs/thigh.stl" scale=" 0.01 0.01 0.01"/>
+            </geometry>
             <material name='black'></material>
-            </geometry>
         </visual>
             <collision>
@@ -270,6 +268,6 @@
             <geometry>
                 <mesh filename="$(find adsmt_description)/adsmt_description/urdf/designs/shin.stl" scale=" 0.01 0.01 0.01"/>
-            <material name='yellow'></material>
-            </geometry>
+            </geometry>
+            <material name='yellow'></material>
         </visual>
             <collision>
@@ -297,6 +295,6 @@
             <geometry>
                 <mesh filename="$(find adsmt_description)/adsmt_description/urdf/designs/double_u_r.stl" scale=" 0.01 0.01 0.01"/>
-            <material name='yellow'></material>
-            </geometry>
+            </geometry>
+            <material name='yellow'></material>
         </visual>
             <collision>
@@ -323,6 +321,6 @@
             <geometry>
                 <mesh filename="$(find adsmt_description)/adsmt_description/urdf/designs/thigh.stl" scale=" 0.01 0.01 0.01"/>
+            </geometry>
             <material name='black'></material>
-            </geometry>
         </visual>
             <collision>
@@ -349,6 +347,6 @@
             <geometry>
                 <mesh filename="$(find adsmt_description)/adsmt_description/urdf/designs/shin.stl" scale=" 0.01 0.01 0.01"/>
-            <material name='yellow'></material>
-            </geometry>
+            </geometry>
+            <material name='yellow'></material>
         </visual>
             <collision>

Commit message: showcase added

File: adsmt_description/adsmt_description/urdf/adsmt.xacro (robot description, xacro)
@@ -6,5 +6,5 @@
     </link>
     <joint name = "body_link_joint" type='fixed'>
-        <origin xyz="0 0 1.5" rpy="0 0 0"/>
+        <origin xyz="0 0 1.5" rpy="0 0 3.1415"/>
         <parent link="base_footprint"/>
         <child link="body"/>
@@ -32,10 +32,10 @@
             <material name='grey'/>
         </visual>
-            <collision>
-               <origin xyz="0 0 0"/>
-               <geometry>
-                  <mesh filename="$(find adsmt_description)/adsmt_description/urdf/designs/body.stl" scale=" 0.01 0.01 0.01"/>
-               </geometry>
-            </collision>
+        <collision>
+           <origin xyz="0 0 0"/>
+           <geometry>
+              <mesh filename="$(find adsmt_description)/adsmt_description/urdf/designs/body.stl" scale=" 0.01 0.01 0.01"/>
+           </geometry>
+        </collision>
     </link>
     <!-- Leg 1 -->
@@ -86,10 +86,10 @@
             <material name='black'></material>
         </visual>
-            <collision>
-                <origin xyz="0 0 0"/>
-                <geometry>
-                    <mesh filename="$(find adsmt_description)/adsmt_description/urdf/designs/thigh.stl" scale=" 0.01 0.01 0.01"/>
-                </geometry>
-            </collision>
+        <collision>
+            <origin xyz="0 0 0"/>
+            <geometry>
+                <mesh filename="$(find adsmt_description)/adsmt_description/urdf/designs/thigh.stl" scale=" 0.01 0.01 0.01"/>
+            </geometry>
+        </collision>
     </link>
     <!-- Shin 1 -->
@@ -113,9 +113,9 @@
             <material name='yellow'></material>
         </visual>
-            <collision>
-                <geometry>
-                    <mesh filename="$(find adsmt_description)/adsmt_description/urdf/designs/shin.stl" scale=" 0.01 0.01 0.01"/>
-                </geometry>
-            </collision>
+        <collision>
+            <geometry>
+                <mesh filename="$(find adsmt_description)/adsmt_description/urdf/designs/shin.stl" scale=" 0.01 0.01 0.01"/>
+            </geometry>
+        </collision>
     </link>
     <!-- /Leg 1 -->
@@ -140,9 +140,9 @@
             <material name='yellow'/>
         </visual>
-            <collision>
-                <geometry>
-                    <mesh filename="$(find adsmt_description)/adsmt_description/urdf/designs/double_u_r.stl" scale=" 0.01 0.01 0.01"/>
-                </geometry>
-            </collision>
+        <collision>
+            <geometry>
+                <mesh filename="$(find adsmt_description)/adsmt_description/urdf/designs/double_u_r.stl" scale=" 0.01 0.01 0.01"/>
+            </geometry>
+        </collision>
     </link>
     <!-- Thigh 2 -->
@@ -166,9 +166,9 @@
             <material name='black'></material>
         </visual>
-            <collision>
-                <geometry>
-                    <mesh filename="$(find adsmt_description)/adsmt_description/urdf/designs/thigh.stl" scale=" 0.01 0.01 0.01"/>
-                </geometry>
-            </collision>
+        <collision>
+            <geometry>
+                <mesh filename="$(find adsmt_description)/adsmt_description/urdf/designs/thigh.stl" scale=" 0.01 0.01 0.01"/>
+            </geometry>
+        </collision>
     </link>
     <!-- Shin 2 -->
@@ -192,9 +192,9 @@
             <material name='yellow'></material>
         </visual>
-            <collision>
-                <geometry>
-                    <mesh filename="$(find adsmt_description)/adsmt_description/urdf/designs/shin.stl" scale=" 0.01 0.01 0.01"/>
-                </geometry>
-            </collision>
+        <collision>
+            <geometry>
+                <mesh filename="$(find adsmt_description)/adsmt_description/urdf/designs/shin.stl" scale=" 0.01 0.01 0.01"/>
+            </geometry>
+        </collision>
     </link>
     <!-- /Leg 2-->
@@ -219,9 +219,9 @@
             <material name='yellow'></material>
         </visual>
-            <collision>
-                <geometry>
-                    <mesh filename="$(find adsmt_description)/adsmt_description/urdf/designs/double_u.stl" scale=" 0.01 0.01 0.01"/>
-                </geometry>
-            </collision>
+        <collision>
+            <geometry>
+                <mesh filename="$(find adsmt_description)/adsmt_description/urdf/designs/double_u.stl" scale=" 0.01 0.01 0.01"/>
+            </geometry>
+        </collision>
     </link>
     <!-- Thigh 3 -->
@@ -245,9 +245,9 @@
             <material name='black'></material>
         </visual>
-            <collision>
-                <geometry>
-                    <mesh filename="$(find adsmt_description)/adsmt_description/urdf/designs/thigh.stl" scale=" 0.01 0.01 0.01"/>
-                </geometry>
-            </collision>
+        <collision>
+            <geometry>
+                <mesh filename="$(find adsmt_description)/adsmt_description/urdf/designs/thigh.stl" scale=" 0.01 0.01 0.01"/>
+            </geometry>
+        </collision>
     </link>
     <!-- Shin 3 -->
@@ -271,9 +271,9 @@
             <material name='yellow'></material>
         </visual>
-            <collision>
-                <geometry>
-                    <mesh filename="$(find adsmt_description)/adsmt_description/urdf/designs/shin.stl" scale=" 0.01 0.01 0.01"/>
-                </geometry>
-            </collision>
+        <collision>
+            <geometry>
+                <mesh filename="$(find adsmt_description)/adsmt_description/urdf/designs/shin.stl" scale=" 0.01 0.01 0.01"/>
+            </geometry>
+        </collision>
     </link>
     <!-- /Leg 3-->
@@ -298,9 +298,9 @@
             <material name='yellow'></material>
         </visual>
-            <collision>
-                <geometry>
-                    <mesh filename="$(find adsmt_description)/adsmt_description/urdf/designs/double_u_r.stl" scale=" 0.01 0.01 0.01"/>
-                </geometry>
-            </collision>
+        <collision>
+            <geometry>
+                <mesh filename="$(find adsmt_description)/adsmt_description/urdf/designs/double_u_r.stl" scale=" 0.01 0.01 0.01"/>
+            </geometry>
+        </collision>
     </link>
     <!-- Thigh 4 -->
@@ -324,9 +324,9 @@
             <material name='black'></material>
         </visual>
-            <collision>
-                <geometry>
-                    <mesh filename="$(find adsmt_description)/adsmt_description/urdf/designs/thigh.stl" scale=" 0.01 0.01 0.01"/>
-                </geometry>
-            </collision>
+        <collision>
+            <geometry>
+                <mesh filename="$(find adsmt_description)/adsmt_description/urdf/designs/thigh.stl" scale=" 0.01 0.01 0.01"/>
+            </geometry>
+        </collision>
     </link>
     <!-- Shin 4 -->
@@ -350,10 +350,9 @@
             <material name='yellow'></material>
         </visual>
-            <collision>
-                <geometry>
-                    <mesh filename="$(find adsmt_description)/adsmt_description/urdf/designs/shin.stl" scale=" 0.01 0.01 0.01"/>
-                    <material name='yellow'></material>
-                </geometry>
-            </collision>
+        <collision>
+            <geometry>
+                <mesh filename="$(find adsmt_description)/adsmt_description/urdf/designs/shin.stl" scale=" 0.01 0.01 0.01"/>
+            </geometry>
+        </collision>
     </link>
     <!-- /Leg 4 -->

Commit message: new strcture

File: adsmt_description/adsmt_description/urdf/adsmt.xacro (robot description, xacro)
@@ -6,5 +6,5 @@
     </link>
     <joint name = "body_link_joint" type='fixed'>
-        <origin xyz="0 0 1.5" rpy="0 0 3.1415"/>
+        <origin xyz="0 0.00 1.5" rpy="0 0 0"/>
         <parent link="base_footprint"/>
         <child link="body"/>
@@ -21,9 +21,4 @@
     <!-- Base Link -->
     <link name="body">
-         <inertial>
-            <mass value="0.29"/>
-            <origin xyz="0 0 0.0"/>
-            <inertia ixx="0.00007" ixy="0.0" ixz="0.0" iyy="0.00007" iyz="0.0" izz="0.00007"/>
-        </inertial>
         <visual>
             <geometry>
@@ -33,4 +28,5 @@
         </visual>
         <collision>
+            <density>1060.0</density>
            <origin xyz="0 0 0"/>
            <geometry>
@@ -38,4 +34,9 @@
            </geometry>
         </collision>
+        <inertial>
+            <mass value="0.29"/>
+            <origin xyz="0 0 0"/>
+            <inertia ixx="0.000193" ixy="0.0" ixz="0.0" iyy="0.000694" iyz="0.0" izz="0.000529"/>
+        </inertial>
     </link>
     <!-- Leg 1 -->
@@ -44,5 +45,5 @@
         <parent link="body"/>
         <child link="joint_1_link"/>
-        <origin xyz="-0.265 -0.60 0.0" rpy="0 0 -1.5708"/>
+        <origin xyz="-0.255 -0.60 0.0" rpy="0 0 -1.5708"/>
         <axis xyz="0 0 1"/>
         <limit lower="-3.1415" upper="3.1415" effort="10" velocity="1.0"/>
@@ -50,7 +51,7 @@
     <link name="joint_1_link">
         <inertial>
-            <mass value="0.04"/>
-            <origin xyz="0 0 0"/>
-            <inertia ixx="0.000005" ixy="0.0" ixz="0.0" iyy="0.000005" iyz="0.0" izz="0.000005"/>
+            <mass value="0.018"/>
+            <origin xyz="0 0 0"/>
+            <inertia ixx="0.000008268" ixy="0.0" ixz="0.0" iyy="0.000008268" iyz="0.0" izz="0.000003468"/>
         </inertial>
         <visual>
@@ -70,5 +71,5 @@
         <parent link="joint_1_link"/>
         <child link="joint_1_thigh"/>
-        <origin xyz="-0.0 -0.46 0.0" rpy="-1.5708 0 0"/>
+        <origin xyz="-0.0 -0.46 -0.0" rpy="-1.5708 0 0"/>
         <axis xyz="1 0 0"/>
         <limit lower="-3.1415" upper="3.1415" effort="10" velocity="1.0"/>
@@ -78,5 +79,5 @@
             <mass value="0.06"/>
             <origin xyz="0 0 0"/>
-            <inertia ixx="0.000005" ixy="0.0" ixz="0.0" iyy="0.000005" iyz="0.0" izz="0.000005"/>
+            <inertia ixx="0.0000193" ixy="0.0" ixz="0.0" iyy="0.0000202" iyz="0.0" izz="0.00000331"/>
         </inertial>
         <visual>
@@ -105,5 +106,5 @@
             <mass value="0.06"/>
             <origin xyz="0 0 0"/>
-            <inertia ixx="0.000005" ixy="0.0" ixz="0.0" iyy="0.000005" iyz="0.0" izz="0.000005"/>
+            <inertia ixx="0.00003064" ixy="0.0" ixz="0" iyy="0.00003232" iyz="0.0" izz="0.0000041"/>
         </inertial>
         <visual>
@@ -124,5 +125,5 @@
         <parent link="body"/>
         <child link="joint_2_link"/>
-        <origin xyz="-0.25 0.6 0.0" rpy="0 0 1.5708"/>
+        <origin xyz="-0.255 0.6 0.0" rpy="0 0 -1.5708"/>
         <axis xyz="0 0 1"/>
         <limit lower="-3.1415" upper="3.1415" effort="10" velocity="1.0"/>
@@ -130,11 +131,11 @@
     <link name="joint_2_link">
         <inertial>
-            <mass value="0.04"/>
-            <origin xyz="0 0 0"/>
-            <inertia ixx="0.000005" ixy="0.0" ixz="0.0" iyy="0.000005" iyz="0.0" izz="0.000005"/>
-        </inertial>
-        <visual>
-            <geometry>
-                <mesh filename="$(find adsmt_description)/adsmt_description/urdf/designs/double_u_r.stl" scale=" 0.01 0.01 0.01"/>
+            <mass value="0.018"/>
+            <origin xyz="0 0 0"/>
+            <inertia ixx="0.000133" ixy="0.0" ixz="0.0" iyy="0.000133" iyz="0.0" izz="0.0000558"/>
+        </inertial>
+        <visual>
+            <geometry>
+                <mesh filename="$(find adsmt_description)/adsmt_description/urdf/designs/double_u.stl" scale=" 0.01 0.01 0.01"/>
             </geometry>
             <material name='yellow'/>
@@ -142,5 +143,5 @@
         <collision>
             <geometry>
-                <mesh filename="$(find adsmt_description)/adsmt_description/urdf/designs/double_u_r.stl" scale=" 0.01 0.01 0.01"/>
+                <mesh filename="$(find adsmt_description)/adsmt_description/urdf/designs/double_u.stl" scale=" 0.01 0.01 0.01"/>
             </geometry>
         </collision>
@@ -150,5 +151,5 @@
         <parent link="joint_2_link"/>
         <child link="joint_2_thigh"/>
-        <origin xyz="-0.0 0.46 0.0" rpy="-1.5708 0 0"/>
+        <origin xyz="-0.0 -0.46 0.0" rpy="-1.5708 0 0"/>
         <axis xyz="1 0 0"/>
         <limit lower="-3.1415" upper="3.1415" effort="10" velocity="1.0"/>
@@ -158,5 +159,5 @@
             <mass value="0.06"/>
             <origin xyz="0 0 0"/>
-            <inertia ixx="0.000005" ixy="0.0" ixz="0.0" iyy="0.000005" iyz="0.0" izz="0.000005"/>
+            <inertia ixx="0.0000193" ixy="0.0" ixz="0.0" iyy="0.0000202" iyz="0.0" izz="0.00000331"/>
         </inertial>
         <visual>
@@ -184,5 +185,5 @@
             <mass value="0.06"/>
             <origin xyz="0 0 0"/>
-            <inertia ixx="0.000005" ixy="0.0" ixz="0.0" iyy="0.000005" iyz="0.0" izz="0.000005"/>
+            <inertia ixx="0.00003064" ixy="0.0" ixz="0" iyy="0.00003232" iyz="0.0" izz="0.0000041"/>
         </inertial>
         <visual>
@@ -203,5 +204,5 @@
         <parent link="body"/>
         <child link="joint_3_link"/>
-        <origin xyz="0.25 -0.60 0.0" rpy="0 0 1.5708"/>
+        <origin xyz="0.25 -0.60 -0.0" rpy="0 0 1.5708"/>
         <axis xyz="0 0 1"/>
         <limit lower="-3.1415" upper="3.1415" effort="10" velocity="1.0"/>
@@ -209,7 +210,7 @@
     <link name="joint_3_link">
         <inertial>
-            <mass value="0.04"/>
-            <origin xyz="0 0 0"/>
-            <inertia ixx="0.000005" ixy="0.0" ixz="0.0" iyy="0.000005" iyz="0.0" izz="0.000005"/>
+            <mass value="0.018"/>
+            <origin xyz="0 0 0"/>
+            <inertia ixx="0.000133" ixy="0.0" ixz="0.0" iyy="0.000133" iyz="0.0" izz="0.0000558"/>
         </inertial>
         <visual>
@@ -229,5 +230,5 @@
         <parent link="joint_3_link"/>
         <child link="joint_3_thigh"/>
-        <origin xyz="-0.0 -0.46 0.0" rpy="-1.5708 0 0"/>
+        <origin xyz="-0.00 -0.46 -0.00" rpy="-1.5708 0 0"/>
         <axis xyz="1 0 0"/>
         <limit lower="-3.1415" upper="3.1415" effort="10" velocity="1.0"/>
@@ -237,5 +238,5 @@
             <mass value="0.06"/>
             <origin xyz="0 0 0"/>
-            <inertia ixx="0.000005" ixy="0.0" ixz="0.0" iyy="0.000005" iyz="0.0" izz="0.000005"/>
+            <inertia ixx="0.0000193" ixy="0.0" ixz="0.0" iyy="0.0000202" iyz="0.0" izz="0.00000331"/>
         </inertial>
         <visual>
@@ -255,5 +256,5 @@
         <parent link="joint_3_thigh"/>
         <child link="joint_3_shin"/>
-        <origin xyz="-0.0 0.65 0.0" rpy="3.1415 0 0"/>
+        <origin xyz="-0.0 0.65 -0.00" rpy="3.1415 0 0"/>
         <axis xyz="1 0 0"/>
         <limit lower="-3.1415" upper="3.1415" effort="10" velocity="1.0"/>
@@ -263,5 +264,5 @@
             <mass value="0.06"/>
             <origin xyz="0 0 0"/>
-            <inertia ixx="0.000005" ixy="0.0" ixz="0.0" iyy="0.000005" iyz="0.0" izz="0.000005"/>
+            <inertia ixx="0.00003064" ixy="0.0" ixz="0" iyy="0.00003232" iyz="0.0" izz="0.0000041"/>
         </inertial>
         <visual>
@@ -282,5 +283,5 @@
         <parent link="body"/>
         <child link="joint_4_link"/>
-        <origin xyz="0.25 0.6 0.0" rpy="0 0 -1.5708"/>
+        <origin xyz="0.250 0.6 0.0" rpy="0 0 1.5708"/>
         <axis xyz="0 0 1"/>
         <limit lower="-3.1415" upper="3.1415" effort="10" velocity="1.0"/>
@@ -288,17 +289,17 @@
     <link name="joint_4_link">
         <inertial>
-            <mass value="0.04"/>
-            <origin xyz="0 0 0"/>
-            <inertia ixx="0.000005" ixy="0.0" ixz="0.0" iyy="0.000005" iyz="0.0" izz="0.000005"/>
-        </inertial>
-        <visual>
-            <geometry>
-                <mesh filename="$(find adsmt_description)/adsmt_description/urdf/designs/double_u_r.stl" scale=" 0.01 0.01 0.01"/>
-            </geometry>
-            <material name='yellow'></material>
-        </visual>
-        <collision>
-            <geometry>
-                <mesh filename="$(find adsmt_description)/adsmt_description/urdf/designs/double_u_r.stl" scale=" 0.01 0.01 0.01"/>
+            <mass value="0.018"/>
+            <origin xyz="0 0 0"/>
+            <inertia ixx="0.000133" ixy="0.0" ixz="0.0" iyy="0.000133" iyz="0.0" izz="0.0000558"/>
+        </inertial>
+        <visual>
+            <geometry>
+                <mesh filename="$(find adsmt_description)/adsmt_description/urdf/designs/double_u.stl" scale=" 0.01 0.01 0.01"/>
+            </geometry>
+            <material name='yellow'></material>
+        </visual>
+        <collision>
+            <geometry>
+                <mesh filename="$(find adsmt_description)/adsmt_description/urdf/designs/double_u.stl" scale=" 0.01 0.01 0.01"/>
             </geometry>
         </collision>
@@ -308,5 +309,5 @@
         <parent link="joint_4_link"/>
         <child link="joint_4_thigh"/>
-        <origin xyz="-0.0 0.46 0.0" rpy="-1.5708 0 0"/>
+        <origin xyz="-0.0 -0.46 0.0" rpy="-1.5708 0 0"/>
         <axis xyz="1 0 0"/>
         <limit lower="-3.1415" upper="3.1415" effort="10" velocity="1.0"/>
@@ -316,5 +317,5 @@
             <mass value="0.06"/>
             <origin xyz="0 0 0"/>
-            <inertia ixx="0.000005" ixy="0.0" ixz="0.0" iyy="0.000005" iyz="0.0" izz="0.000005"/>
+            <inertia ixx="0.0000193" ixy="0.0" ixz="0.0" iyy="0.0000202" iyz="0.0" izz="0.00000331"/>
         </inertial>
         <visual>
@@ -342,5 +343,5 @@
             <mass value="0.06"/>
             <origin xyz="0 0 0"/>
-            <inertia ixx="0.000005" ixy="0.0" ixz="0.0" iyy="0.000005" iyz="0.0" izz="0.000005"/>
+            <inertia ixx="0.00003064" ixy="0.0" ixz="0" iyy="0.00003232" iyz="0.0" izz="0.0000041"/>
         </inertial>
         <visual>
