Commit message: added drive functionalities

File: adsmt_description/adsmt_description/urdf/adsmt-wheeled.xacro (robot description, xacro)
@@ -1,10 +1,10 @@
 <?xml version="1.0" ?>
 <robot name="ads-mt" xmlns:xacro="http://www.ros.org/wiki/xacro">
-    <xacro:include filename="$(find adsmt_description)/adsmt_description/urdf/adsmt.gazebo" />
+    <xacro:include filename="$(find adsmt_description)/adsmt_description/urdf/adsmt-wheeled.gazebo" />
     <link name = "base_footprint">
         <!-- Nth in here -->
     </link>
     <joint name = "body_link_joint" type='fixed'>
-        <origin xyz="0 0.00 1.5" rpy="0 0 0"/>
+        <origin xyz="0 0.00 1.565" rpy="0 0 0"/>
         <parent link="base_footprint"/>
         <child link="body"/>
@@ -120,4 +120,31 @@
         </collision>
     </link>
+    <!-- Wheel 1 -->
+    <joint name="wheel_1" type="continuous">
+        <parent link="joint_1_shin"/>
+        <child link="joint_1_wheel"/>
+        <origin xyz="0.18 -0.65 0.0" rpy="1.5708 0 1.5708"/>
+        <axis xyz="0 0 1"/>
+        <dynamics damping="0.01" friction='1.0' />
+        <limit lower="-3.1415" upper="3.1415" effort="150" velocity="50.0"/>
+    </joint>
+    <link name="joint_1_wheel">
+        <inertial>
+            <mass value="0.06"/>
+            <origin xyz="0 0 0"/>
+            <inertia ixx="0.000135" ixy="0.0" ixz="0" iyy="0.000135" iyz="0.0" izz="0.000265"/>
+        </inertial>
+        <visual>
+            <geometry>
+                <cylinder radius="0.23" length = "0.055"/>
+            </geometry>
+            <material name='black'></material>
+        </visual>
+        <collision>
+            <geometry>
+                <cylinder radius="0.23" length = "0.055"/>
+            </geometry>
+        </collision>
+    </link>
     <!-- /Leg 1 -->
     <!-- Leg 2 -->
@@ -199,4 +226,31 @@
         </collision>
     </link>
+    <joint name="wheel_2" type="continuous">
+        <parent link="joint_2_shin"/>
+        <child link="joint_2_wheel"/>
+        <origin xyz="-0.18 -0.65 0.0" rpy="1.5708 0 1.5708"/>
+        <dynamics damping="0.01" friction='1.0' />
+        <axis xyz="0 0 1"/>
+        <limit lower="-3.1415" upper="3.1415" effort="150" velocity="50.0"/>
+    </joint>
+    <!-- Wheel 2 -->
+    <link name="joint_2_wheel">
+        <inertial>
+            <mass value="0.06"/>
+            <origin xyz="0 0 0"/>
+            <inertia ixx="0.000135" ixy="0.0" ixz="0" iyy="0.000135" iyz="0.0" izz="0.000265"/>
+        </inertial>
+        <visual>
+            <geometry>
+                <cylinder radius="0.23" length = "0.055"/>
+            </geometry>
+            <material name='black'></material>
+        </visual>
+        <collision>
+            <geometry>
+                <cylinder radius="0.23" length = "0.055"/>
+            </geometry>
+        </collision>
+    </link>
     <!-- /Leg 2-->
     <!-- Leg 3 -->
@@ -278,4 +332,31 @@
         </collision>
     </link>
+    <!-- Wheel 3 -->
+    <joint name="wheel_3" type="continuous">
+        <parent link="joint_3_shin"/>
+        <dynamics damping="0.01" friction='1.0' />
+        <child link="joint_3_wheel"/>
+        <origin xyz="-0.18 -0.65 0.0" rpy="1.5708 0 1.5708"/>
+        <axis xyz="0 0 1"/>
+        <limit lower="-3.1415" upper="3.1415" effort="150" velocity="50.0"/>
+    </joint>
+    <link name="joint_3_wheel">
+        <inertial>
+            <mass value="0.06"/>
+            <origin xyz="0 0 0"/>
+            <inertia ixx="0.000135" ixy="0.0" ixz="0" iyy="0.000135" iyz="0.0" izz="0.000265"/>
+        </inertial>
+        <visual>
+            <geometry>
+                <cylinder radius="0.23" length = "0.055"/>
+            </geometry>
+            <material name='black'></material>
+        </visual>
+        <collision>
+            <geometry>
+                <cylinder radius="0.23" length = "0.055"/>
+            </geometry>
+        </collision>
+    </link>
     <!-- /Leg 3-->
     <!-- Leg 4 -->
@@ -357,4 +438,31 @@
         </collision>
     </link>
+    <!-- Wheel 4 -->
+    <joint name="wheel_4" type="continuous">
+        <parent link="joint_4_shin"/>
+        <dynamics damping="0.01" friction='1.0' />
+        <child link="joint_4_wheel"/>
+        <origin xyz="0.18 -0.65 0.0" rpy="1.5708 0 1.5708"/>
+        <axis xyz="0 0 1"/>
+        <limit lower="-3.1415" upper="3.1415" effort="150" velocity="50.0"/>
+    </joint>
+    <link name="joint_4_wheel">
+        <inertial>
+            <mass value="0.06"/>
+            <origin xyz="0 0 0"/>
+            <inertia ixx="0.000135" ixy="0.0" ixz="0" iyy="0.000135" iyz="0.0" izz="0.000265"/>
+        </inertial>
+        <visual>
+            <geometry>
+                <cylinder radius="0.23" length = "0.055"/>
+            </geometry>
+            <material name='black'></material>
+        </visual>
+        <collision>
+            <geometry>
+                <cylinder radius="0.23" length = "0.055"/>
+            </geometry>
+        </collision>
+    </link>
     <!-- /Leg 4 -->
 </robot>
