Commit message: added odometry

File: adsmt_description/adsmt_description/urdf/adsmt-wheeled.xacro (robot description, xacro)
@@ -6,5 +6,5 @@
     </link>
     <joint name = "body_link_joint" type='fixed'>
-        <origin xyz="0 0.00 1.565" rpy="0 0 0"/>
+        <origin xyz="0 0.00 0.1565" rpy="0 0 0"/>
         <parent link="base_footprint"/>
         <child link="body"/>
@@ -23,5 +23,5 @@
         <visual>
             <geometry>
-                <mesh filename="$(find adsmt_description)/adsmt_description/urdf/designs/body.stl" scale=" 0.01 0.01 0.01"/>
+                <mesh filename="$(find adsmt_description)/adsmt_description/urdf/designs/body.stl" scale=" 0.001 0.001 0.001"/>
             </geometry>
             <material name='grey'/>
@@ -31,5 +31,5 @@
            <origin xyz="0 0 0"/>
            <geometry>
-              <mesh filename="$(find adsmt_description)/adsmt_description/urdf/designs/body.stl" scale=" 0.01 0.01 0.01"/>
+              <mesh filename="$(find adsmt_description)/adsmt_description/urdf/designs/body.stl" scale=" 0.001 0.001 0.001"/>
            </geometry>
         </collision>
@@ -45,5 +45,5 @@
         <parent link="body"/>
         <child link="joint_1_link"/>
-        <origin xyz="-0.255 -0.60 0.0" rpy="0 0 -1.5708"/>
+        <origin xyz="-0.0255 -0.060 0.0" rpy="0 0 -1.5708"/>
         <axis xyz="0 0 1"/>
         <limit lower="-3.1415" upper="3.1415" effort="50" velocity="2.0"/>
@@ -57,5 +57,5 @@
         <visual>
             <geometry>
-                <mesh filename="$(find adsmt_description)/adsmt_description/urdf/designs/double_u.stl" scale=" 0.01 0.01 0.01"/>
+                <mesh filename="$(find adsmt_description)/adsmt_description/urdf/designs/double_u.stl" scale=" 0.001 0.001 0.001"/>
             </geometry>
             <material name='yellow'/>
@@ -63,5 +63,5 @@
         <collision>
             <geometry>
-                <mesh filename="$(find adsmt_description)/adsmt_description/urdf/designs/double_u.stl" scale=" 0.01 0.01 0.01"/>
+                <mesh filename="$(find adsmt_description)/adsmt_description/urdf/designs/double_u.stl" scale=" 0.001 0.001 0.001"/>
             </geometry>
         </collision>
@@ -71,5 +71,5 @@
         <parent link="joint_1_link"/>
         <child link="joint_1_thigh"/>
-        <origin xyz="-0.0 -0.46 -0.0" rpy="-1.5708 0 0"/>
+        <origin xyz="-0.0 -0.046 -0.0" rpy="-1.5708 0 0"/>
         <axis xyz="1 0 0"/>
         <limit lower="-3.1415" upper="3.1415" effort="50" velocity="2.0"/>
@@ -83,12 +83,12 @@
         <visual>
             <geometry>
-                <mesh filename="$(find adsmt_description)/adsmt_description/urdf/designs/thigh.stl" scale=" 0.01 0.01 0.01"/>
-            </geometry>
-            <material name='black'></material>
-        </visual>
-        <collision>
-            <origin xyz="0 0 0"/>
-            <geometry>
-                <mesh filename="$(find adsmt_description)/adsmt_description/urdf/designs/thigh.stl" scale=" 0.01 0.01 0.01"/>
+                <mesh filename="$(find adsmt_description)/adsmt_description/urdf/designs/thigh.stl" scale=" 0.001 0.001 0.001"/>
+            </geometry>
+            <material name='black'></material>
+        </visual>
+        <collision>
+            <origin xyz="0 0 0"/>
+            <geometry>
+                <mesh filename="$(find adsmt_description)/adsmt_description/urdf/designs/thigh.stl" scale=" 0.001 0.001 0.001"/>
             </geometry>
         </collision>
@@ -98,5 +98,5 @@
         <parent link="joint_1_thigh"/>
         <child link="joint_1_shin"/>
-        <origin xyz="-0.0 0.65 0.0" rpy="3.1415 0 0"/>
+        <origin xyz="-0.0 0.065 0.0" rpy="3.1415 0 0"/>
         <axis xyz="1 0 0"/>
         <limit lower="-3.1415" upper="3.1415" effort="50" velocity="2.0"/>
@@ -110,11 +110,11 @@
         <visual>
             <geometry>
-                <mesh filename="$(find adsmt_description)/adsmt_description/urdf/designs/shin.stl" scale=" 0.01 0.01 0.01"/>
-            </geometry>
-            <material name='yellow'></material>
-        </visual>
-        <collision>
-            <geometry>
-                <mesh filename="$(find adsmt_description)/adsmt_description/urdf/designs/shin.stl" scale=" 0.01 0.01 0.01"/>
+                <mesh filename="$(find adsmt_description)/adsmt_description/urdf/designs/shin.stl" scale=" 0.001 0.001 0.001"/>
+            </geometry>
+            <material name='yellow'></material>
+        </visual>
+        <collision>
+            <geometry>
+                <mesh filename="$(find adsmt_description)/adsmt_description/urdf/designs/shin.stl" scale=" 0.001 0.001 0.001"/>
             </geometry>
         </collision>
@@ -124,5 +124,5 @@
         <parent link="joint_1_shin"/>
         <child link="joint_1_wheel"/>
-        <origin xyz="0.18 -0.65 0.0" rpy="1.5708 0 1.5708"/>
+        <origin xyz="0.018 -0.065 0.0" rpy="1.5708 0 1.5708"/>
         <axis xyz="0 0 1"/>
         <dynamics damping="0.01" friction='1.0' />
@@ -137,11 +137,11 @@
         <visual>
             <geometry>
-                <cylinder radius="0.23" length = "0.055"/>
-            </geometry>
-            <material name='black'></material>
-        </visual>
-        <collision>
-            <geometry>
-                <cylinder radius="0.23" length = "0.055"/>
+                <cylinder radius="0.023" length = "0.0055"/>
+            </geometry>
+            <material name='black'></material>
+        </visual>
+        <collision>
+            <geometry>
+                <cylinder radius="0.023" length = "0.0055"/>
             </geometry>
         </collision>
@@ -152,5 +152,5 @@
         <parent link="body"/>
         <child link="joint_2_link"/>
-        <origin xyz="-0.255 0.6 0.0" rpy="0 0 -1.5708"/>
+        <origin xyz="-0.0255 0.06 0.0" rpy="0 0 -1.5708"/>
         <axis xyz="0 0 1"/>
         <limit lower="-3.1415" upper="3.1415" effort="50" velocity="2.0"/>
@@ -164,5 +164,5 @@
         <visual>
             <geometry>
-                <mesh filename="$(find adsmt_description)/adsmt_description/urdf/designs/double_u.stl" scale=" 0.01 0.01 0.01"/>
+                <mesh filename="$(find adsmt_description)/adsmt_description/urdf/designs/double_u.stl" scale=" 0.001 0.001 0.001"/>
             </geometry>
             <material name='yellow'/>
@@ -170,5 +170,5 @@
         <collision>
             <geometry>
-                <mesh filename="$(find adsmt_description)/adsmt_description/urdf/designs/double_u.stl" scale=" 0.01 0.01 0.01"/>
+                <mesh filename="$(find adsmt_description)/adsmt_description/urdf/designs/double_u.stl" scale=" 0.001 0.001 0.001"/>
             </geometry>
         </collision>
@@ -178,5 +178,5 @@
         <parent link="joint_2_link"/>
         <child link="joint_2_thigh"/>
-        <origin xyz="-0.0 -0.46 0.0" rpy="-1.5708 0 0"/>
+        <origin xyz="-0.0 -0.046 0.0" rpy="-1.5708 0 0"/>
         <axis xyz="1 0 0"/>
         <limit lower="-3.1415" upper="3.1415" effort="50" velocity="2.0"/>
@@ -190,11 +190,11 @@
         <visual>
             <geometry>
-                <mesh filename="$(find adsmt_description)/adsmt_description/urdf/designs/thigh.stl" scale=" 0.01 0.01 0.01"/>
-            </geometry>
-            <material name='black'></material>
-        </visual>
-        <collision>
-            <geometry>
-                <mesh filename="$(find adsmt_description)/adsmt_description/urdf/designs/thigh.stl" scale=" 0.01 0.01 0.01"/>
+                <mesh filename="$(find adsmt_description)/adsmt_description/urdf/designs/thigh.stl" scale=" 0.001 0.001 0.001"/>
+            </geometry>
+            <material name='black'></material>
+        </visual>
+        <collision>
+            <geometry>
+                <mesh filename="$(find adsmt_description)/adsmt_description/urdf/designs/thigh.stl" scale=" 0.001 0.001 0.001"/>
             </geometry>
         </collision>
@@ -204,5 +204,5 @@
         <parent link="joint_2_thigh"/>
         <child link="joint_2_shin"/>
-        <origin xyz="-0.0 0.65 0.0" rpy="3.1415 0 0"/>
+        <origin xyz="-0.0 0.065 0.0" rpy="3.1415 0 0"/>
         <axis xyz="1 0 0"/>
         <limit lower="-3.1415" upper="3.1415" effort="50" velocity="2.0"/>
@@ -216,11 +216,11 @@
         <visual>
             <geometry>
-                <mesh filename="$(find adsmt_description)/adsmt_description/urdf/designs/shin.stl" scale=" 0.01 0.01 0.01"/>
-            </geometry>
-            <material name='yellow'></material>
-        </visual>
-        <collision>
-            <geometry>
-                <mesh filename="$(find adsmt_description)/adsmt_description/urdf/designs/shin.stl" scale=" 0.01 0.01 0.01"/>
+                <mesh filename="$(find adsmt_description)/adsmt_description/urdf/designs/shin.stl" scale=" 0.001 0.001 0.001"/>
+            </geometry>
+            <material name='yellow'></material>
+        </visual>
+        <collision>
+            <geometry>
+                <mesh filename="$(find adsmt_description)/adsmt_description/urdf/designs/shin.stl" scale=" 0.001 0.001 0.001"/>
             </geometry>
         </collision>
@@ -229,5 +229,5 @@
         <parent link="joint_2_shin"/>
         <child link="joint_2_wheel"/>
-        <origin xyz="-0.18 -0.65 0.0" rpy="1.5708 0 1.5708"/>
+        <origin xyz="-0.018 -0.065 0.0" rpy="1.5708 0 1.5708"/>
         <dynamics damping="0.01" friction='1.0' />
         <axis xyz="0 0 1"/>
@@ -243,11 +243,11 @@
         <visual>
             <geometry>
-                <cylinder radius="0.23" length = "0.055"/>
-            </geometry>
-            <material name='black'></material>
-        </visual>
-        <collision>
-            <geometry>
-                <cylinder radius="0.23" length = "0.055"/>
+                <cylinder radius="0.023" length = "0.0055"/>
+            </geometry>
+            <material name='black'></material>
+        </visual>
+        <collision>
+            <geometry>
+                <cylinder radius="0.023" length = "0.0055"/>
             </geometry>
         </collision>
@@ -258,5 +258,5 @@
         <parent link="body"/>
         <child link="joint_3_link"/>
-        <origin xyz="0.25 -0.60 -0.0" rpy="0 0 1.5708"/>
+        <origin xyz="0.025 -0.060 -0.0" rpy="0 0 1.5708"/>
         <axis xyz="0 0 1"/>
         <limit lower="-3.1415" upper="3.1415" effort="50" velocity="2.0"/>
@@ -270,11 +270,11 @@
         <visual>
             <geometry>
-                <mesh filename="$(find adsmt_description)/adsmt_description/urdf/designs/double_u.stl" scale=" 0.01 0.01 0.01"/>
-            </geometry>
-            <material name='yellow'></material>
-        </visual>
-        <collision>
-            <geometry>
-                <mesh filename="$(find adsmt_description)/adsmt_description/urdf/designs/double_u.stl" scale=" 0.01 0.01 0.01"/>
+                <mesh filename="$(find adsmt_description)/adsmt_description/urdf/designs/double_u.stl" scale=" 0.001 0.001 0.001"/>
+            </geometry>
+            <material name='yellow'></material>
+        </visual>
+        <collision>
+            <geometry>
+                <mesh filename="$(find adsmt_description)/adsmt_description/urdf/designs/double_u.stl" scale=" 0.001 0.001 0.001"/>
             </geometry>
         </collision>
@@ -284,5 +284,5 @@
         <parent link="joint_3_link"/>
         <child link="joint_3_thigh"/>
-        <origin xyz="-0.00 -0.46 -0.00" rpy="-1.5708 0 0"/>
+        <origin xyz="-0.00 -0.046 -0.00" rpy="-1.5708 0 0"/>
         <axis xyz="1 0 0"/>
         <limit lower="-3.1415" upper="3.1415" effort="50" velocity="2.0"/>
@@ -296,11 +296,11 @@
         <visual>
             <geometry>
-                <mesh filename="$(find adsmt_description)/adsmt_description/urdf/designs/thigh.stl" scale=" 0.01 0.01 0.01"/>
-            </geometry>
-            <material name='black'></material>
-        </visual>
-        <collision>
-            <geometry>
-                <mesh filename="$(find adsmt_description)/adsmt_description/urdf/designs/thigh.stl" scale=" 0.01 0.01 0.01"/>
+                <mesh filename="$(find adsmt_description)/adsmt_description/urdf/designs/thigh.stl" scale=" 0.001 0.001 0.001"/>
+            </geometry>
+            <material name='black'></material>
+        </visual>
+        <collision>
+            <geometry>
+                <mesh filename="$(find adsmt_description)/adsmt_description/urdf/designs/thigh.stl" scale=" 0.001 0.001 0.001"/>
             </geometry>
         </collision>
@@ -310,5 +310,5 @@
         <parent link="joint_3_thigh"/>
         <child link="joint_3_shin"/>
-        <origin xyz="-0.0 0.65 -0.00" rpy="3.1415 0 0"/>
+        <origin xyz="-0.0 0.065 -0.00" rpy="3.1415 0 0"/>
         <axis xyz="1 0 0"/>
         <limit lower="-3.1415" upper="3.1415" effort="50" velocity="2.0"/>
@@ -322,11 +322,11 @@
         <visual>
             <geometry>
-                <mesh filename="$(find adsmt_description)/adsmt_description/urdf/designs/shin.stl" scale=" 0.01 0.01 0.01"/>
-            </geometry>
-            <material name='yellow'></material>
-        </visual>
-        <collision>
-            <geometry>
-                <mesh filename="$(find adsmt_description)/adsmt_description/urdf/designs/shin.stl" scale=" 0.01 0.01 0.01"/>
+                <mesh filename="$(find adsmt_description)/adsmt_description/urdf/designs/shin.stl" scale=" 0.001 0.001 0.001"/>
+            </geometry>
+            <material name='yellow'></material>
+        </visual>
+        <collision>
+            <geometry>
+                <mesh filename="$(find adsmt_description)/adsmt_description/urdf/designs/shin.stl" scale=" 0.001 0.001 0.001"/>
             </geometry>
         </collision>
@@ -337,5 +337,5 @@
         <dynamics damping="0.01" friction='1.0' />
         <child link="joint_3_wheel"/>
-        <origin xyz="-0.18 -0.65 0.0" rpy="1.5708 0 1.5708"/>
+        <origin xyz="-0.018 -0.065 0.0" rpy="1.5708 0 1.5708"/>
         <axis xyz="0 0 1"/>
         <limit lower="-3.1415" upper="3.1415" effort="150" velocity="50.0"/>
@@ -349,11 +349,11 @@
         <visual>
             <geometry>
-                <cylinder radius="0.23" length = "0.055"/>
-            </geometry>
-            <material name='black'></material>
-        </visual>
-        <collision>
-            <geometry>
-                <cylinder radius="0.23" length = "0.055"/>
+                <cylinder radius="0.023" length = "0.0055"/>
+            </geometry>
+            <material name='black'></material>
+        </visual>
+        <collision>
+            <geometry>
+                <cylinder radius="0.023" length = "0.0055"/>
             </geometry>
         </collision>
@@ -364,5 +364,5 @@
         <parent link="body"/>
         <child link="joint_4_link"/>
-        <origin xyz="0.250 0.6 0.0" rpy="0 0 1.5708"/>
+        <origin xyz="0.0250 0.06 0.0" rpy="0 0 1.5708"/>
         <axis xyz="0 0 1"/>
         <limit lower="-3.1415" upper="3.1415" effort="50" velocity="2.0"/>
@@ -376,11 +376,11 @@
         <visual>
             <geometry>
-                <mesh filename="$(find adsmt_description)/adsmt_description/urdf/designs/double_u.stl" scale=" 0.01 0.01 0.01"/>
-            </geometry>
-            <material name='yellow'></material>
-        </visual>
-        <collision>
-            <geometry>
-                <mesh filename="$(find adsmt_description)/adsmt_description/urdf/designs/double_u.stl" scale=" 0.01 0.01 0.01"/>
+                <mesh filename="$(find adsmt_description)/adsmt_description/urdf/designs/double_u.stl" scale=" 0.001 0.001 0.001"/>
+            </geometry>
+            <material name='yellow'></material>
+        </visual>
+        <collision>
+            <geometry>
+                <mesh filename="$(find adsmt_description)/adsmt_description/urdf/designs/double_u.stl" scale=" 0.001 0.001 0.001"/>
             </geometry>
         </collision>
@@ -390,5 +390,5 @@
         <parent link="joint_4_link"/>
         <child link="joint_4_thigh"/>
-        <origin xyz="-0.0 -0.46 0.0" rpy="-1.5708 0 0"/>
+        <origin xyz="-0.0 -0.046 0.0" rpy="-1.5708 0 0"/>
         <axis xyz="1 0 0"/>
         <limit lower="-3.1415" upper="3.1415" effort="50" velocity="2.0"/>
@@ -402,11 +402,11 @@
         <visual>
             <geometry>
-                <mesh filename="$(find adsmt_description)/adsmt_description/urdf/designs/thigh.stl" scale=" 0.01 0.01 0.01"/>
-            </geometry>
-            <material name='black'></material>
-        </visual>
-        <collision>
-            <geometry>
-                <mesh filename="$(find adsmt_description)/adsmt_description/urdf/designs/thigh.stl" scale=" 0.01 0.01 0.01"/>
+                <mesh filename="$(find adsmt_description)/adsmt_description/urdf/designs/thigh.stl" scale=" 0.001 0.001 0.001"/>
+            </geometry>
+            <material name='black'></material>
+        </visual>
+        <collision>
+            <geometry>
+                <mesh filename="$(find adsmt_description)/adsmt_description/urdf/designs/thigh.stl" scale=" 0.001 0.001 0.001"/>
             </geometry>
         </collision>
@@ -416,5 +416,5 @@
         <parent link="joint_4_thigh"/>
         <child link="joint_4_shin"/>
-        <origin xyz="-0.0 0.65 0.0" rpy="3.1415 0 0"/>
+        <origin xyz="-0.0 0.065 0.0" rpy="3.1415 0 0"/>
         <axis xyz="1 0 0"/>
         <limit lower="-3.1415" upper="3.1415" effort="50" velocity="2.0"/>
@@ -428,11 +428,11 @@
         <visual>
             <geometry>
-                <mesh filename="$(find adsmt_description)/adsmt_description/urdf/designs/shin.stl" scale=" 0.01 0.01 0.01"/>
-            </geometry>
-            <material name='yellow'></material>
-        </visual>
-        <collision>
-            <geometry>
-                <mesh filename="$(find adsmt_description)/adsmt_description/urdf/designs/shin.stl" scale=" 0.01 0.01 0.01"/>
+                <mesh filename="$(find adsmt_description)/adsmt_description/urdf/designs/shin.stl" scale=" 0.001 0.001 0.001"/>
+            </geometry>
+            <material name='yellow'></material>
+        </visual>
+        <collision>
+            <geometry>
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